File: badge-kit.kicad_pcb (KiCad board)
At the start: 2 copper layers, 38 x 48.9 mm, 13 parts, among them SW1 BYPASS SWITCH >, SW2 OFF/ON, SW2 ON/OFF, SW3 < BYPASS RESISTOR

Commit message: Updated PCB
Parts:
- turned SW1 to 310 degrees
Routing:
- net Net-(R1-Pad1): track 52.8 -> 95.2 mm
- net GND: track 9.93 -> 35.6 mm
- net Net-(BT1-Pad1): track 40.4 -> 23.5 mm
Other:
- board text added: "+"
- board text added: "-"
