File: Coffs Harbour Rocket/badge-kit.kicad_pcb (KiCad board)
At the start: 2 copper layers, 38 x 48.9 mm, 7 parts, among them J1 LOGO, J2 LOGO_SMALL, SW2 ON/OFF

Commit message: Updated PCBS
Parts:
- SW2: value ON/OFF -> OFF/ON
Changed lines of the file:
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@@
   )
   (setup
-    (last_trace_width 1)
+    (last_trace_width 0.25)
     (user_trace_width 0.25)
     (user_trace_width 0.5)
@@
       (effects (font (size 0.8 0.8) (thickness 0.12)) (justify mirror))
     )
-    (fp_text value ON/OFF (at 0.10396 2.567507 130) (layer B.SilkS)
+    (fp_text value OFF/ON (at 0.10396 2.567507 130) (layer B.SilkS)
       (effects (font (size 1 1) (thickness 0.15)) (justify mirror))
     )
