File: Multimeter Ruler/Multimeter-Ruler.sch (KiCad schematic (older format))
At the start: 27 parts

Commit message: Schematic ready for PCB design
Parts:
- BT1: renamed from BT?; footprint (none) -> libs:CR2032
- C1, C10, C11, C2, C3, C4, C5, C6, C7, C8, C9: renamed from C?; footprint (none) -> Capacitors_SMD:C_0603_HandSoldering
- J1, J2: renamed from J?; footprint (none) -> Pin_Headers:Pin_Header_Angled_1x01_Pitch2.54mm
- J3: renamed from J?; footprint (none) -> Pin_Headers:Pin_Header_Straight_2x03_Pitch2.54mm
- LS1: renamed from LS?; footprint (none) -> libs:hyg7525
- R1, R2, R3, R4, R5, R6: renamed from R?; footprint (none) -> Resistors_SMD:R_0603_HandSoldering
- SW2: renamed from SW?; footprint (none) -> libs:SS12D00
- U2: renamed from U?; footprint (none) -> libs:NHD-C12832A1Z
- Y1: renamed from Y?; footprint (none) -> Crystals:Crystal_SMD_0603-4pin_6.0x3.5mm_HandSoldering
- gave numbers to parts that had none: 2

Commit message: Added PCB
Parts:
- removed Y1: 16MHz, Crystals:Crystal_SMD_0603-4pin_6.0x3.5mm_HandSoldering, symbol Crystal
- added J4: MECH, Mounting_Holes:MountingHole_5.3mm_M5, symbol Conn_01x01
- added Y1: Crystal_GND24, Crystals:Crystal_SMD_3225-4pin_3.2x2.5mm_HandSoldering, symbol Crystal_GND24
- BT1: value Battery_Cell -> CR2102
- SW1: footprint (none) -> libs:1107G
Connections:
- net +3V3: no longer U2.A
- net GND: now also Y1.2, Y1.4
- net D9: now reaches U1.13 ((OC1A/PTCXY)PB1)
- net D9: now also U2.A
- net at C2.1, R4.1, U1.7 ((XTAL1/TOSC1)PB6): now also Y1.1
- net at C3.1, R4.2, U1.8 ((XTAL2/TOSC2)PB7): now also Y1.3
- no-connect marks 2 -> 18
Other:
- moved on the sheet: C2, C3
Changed lines of the file:
@@
 LIBS:valves
 LIBS:nhd-c12832a1z
-LIBS:crystal_4pin_smd
 LIBS:Multimeter-Ruler-cache
 EELAYER 25 0
@@
 P 1000 1300
 F 0 "BT1" H 1100 1400 50  0000 L CNN
-F 1 "Battery_Cell" H 1100 1300 50  0000 L CNN
+F 1 "CR2102" H 1100 1300 50  0000 L CNN
 F 2 "libs:CR2032" V 1000 1360 50  0001 C CNN
 F 3 "" V 1000 1360 50  0001 C CNN
@@
 $EndComp
 $Comp
-L GND #PWR01
+L GND #PWR1
 U 1 1 5B17DD9B
 P 1000 1500
-F 0 "#PWR01" H 1000 1250 50  0001 C CNN
+F 0 "#PWR1" H 1000 1250 50  0001 C CNN
 F 1 "GND" H 1000 1350 50  0000 C CNN
 F 2 "" H 1000 1500 50  0001 C CNN
@@
 $EndComp
 $Comp
-L +3.3V #PWR02
+L +3.3V #PWR8
 U 1 1 5B17DDB1
 P 2700 800
-F 0 "#PWR02" H 2700 650 50  0001 C CNN
+F 0 "#PWR8" H 2700 650 50  0001 C CNN
 F 1 "+3.3V" H 2700 940 50  0000 C CNN
 F 2 "" H 2700 800 50  0001 C CNN
@@
 	1000 1100 1000 1000
 $Comp
-L +3.3V #PWR03
-U 1 1 5B17E239
-P 4850 1100
-F 0 "#PWR03" H 4850 950 50  0001 C CNN
-F 1 "+3.3V" H 4850 1240 50  0000 C CNN
-F 2 "" H 4850 1100 50  0001 C CNN
-F 3 "" H 4850 1100 50  0001 C CNN
-	1    4850 1100
-	1    0    0    -1
-$EndComp
-$Comp
-L GND #PWR04
+L GND #PWR12
 U 1 1 5B17E24A
 P 4850 1400
-F 0 "#PWR04" H 4850 1150 50  0001 C CNN
+F 0 "#PWR12" H 4850 1150 50  0001 C CNN
 F 1 "GND" H 4850 1250 50  0000 C CNN
 F 2 "" H 4850 1400 50  0001 C CNN
@@
 $EndComp
 Wire Wire Line
-	4850 1100 4850 1150
-Wire Wire Line
-	4850 1150 4900 1150
+	4700 1150 4900 1150
 Wire Wire Line
 	4850 1400 4850 1350
@@
 	4850 1350 4900 1350
 $Comp
-L GND #PWR05
+L GND #PWR15
 U 1 1 5B17E620
 P 6400 2650
-F 0 "#PWR05" H 6400 2400 50  0001 C CNN
+F 0 "#PWR15" H 6400 2400 50  0001 C CNN
 F 1 "GND" H 6400 2500 50  0000 C CNN
 F 2 "" H 6400 2650 50  0001 C CNN
@@
 $EndComp
 $Comp
-L +3.3V #PWR06
+L +3.3V #PWR14
 U 1 1 5B17E631
 P 6250 2400
-F 0 "#PWR06" H 6250 2250 50  0001 C CNN
+F 0 "#PWR14" H 6250 2250 50  0001 C CNN
 F 1 "+3.3V" H 6250 2540 50  0000 C CNN
 F 2 "" H 6250 2400 50  0001 C CNN
@@
 Connection ~ 6400 2600
 $Comp
-L GND #PWR07
+L GND #PWR17
 U 1 1 5B17E7E7
 P 8300 1750
-F 0 "#PWR07" H 8300 1500 50  0001 C CNN
+F 0 "#PWR17" H 8300 1500 50  0001 C CNN
 F 1 "GND" H 8300 1600 50  0000 C CNN
 F 2 "" H 8300 1750 50  0001 C CNN
@@
 	4200 5550 3700 5550
 $Comp
-L GND #PWR08
+L GND #PWR7
 U 1 1 5B18104A
 P 2300 7450
-F 0 "#PWR08" H 2300 7200 50  0001 C CNN
+F 0 "#PWR7" H 2300 7200 50  0001 C CNN
 F 1 "GND" H 2300 7300 50  0000 C CNN
 F 2 "" H 2300 7450 50  0001 C CNN
@@
 $EndComp
 $Comp
-L +3.3V #PWR09
+L +3.3V #PWR18
 U 1 1 5B1813F0
 P 10300 1250
-F 0 "#PWR09" H 10300 1100 50  0001 C CNN
+F 0 "#PWR18" H 10300 1100 50  0001 C CNN
 F 1 "+3.3V" H 10300 1390 50  0000 C CNN
 F 2 "" H 10300 1250 50  0001 C CNN
@@
 $EndComp
 $Comp
-L GND #PWR010
+L GND #PWR19
 U 1 1 5B1814DF
 P 10300 1550
-F 0 "#PWR010" H 10300 1300 50  0001 C CNN
+F 0 "#PWR19" H 10300 1300 50  0001 C CNN
 F 1 "GND" H 10300 1400 50  0000 C CNN
 F 2 "" H 10300 1550 50  0001 C CNN
@@
 F 0 "SW1" H 1650 2950 50  0000 L CNN
 F 1 "TOGGLE" H 1600 2790 50  0000 C CNN
-F 2 "" H 1600 3050 50  0001 C CNN
+F 2 "libs:1107G" H 1600 3050 50  0001 C CNN
 F 3 "" H 1600 3050 50  0001 C CNN
 	1    1600 2850
@@
 $EndComp
 $Comp
-L +3.3V #PWR011
+L +3.3V #PWR6
 U 1 1 5B1823FD
 P 2300 4250
-F 0 "#PWR011" H 2300 4100 50  0001 C CNN
+F 0 "#PWR6" H 2300 4100 50  0001 C CNN
 F 1 "+3.3V" H 2300 4390 50  0000 C CNN
 F 2 "" H 2300 4250 50  0001 C CNN
@@
 NoConn ~ 1100 4950
 $Comp
-L +3.3V #PWR012
+L +3.3V #PWR2
 U 1 1 5B182683
 P 1000 5400
-F 0 "#PWR012" H 1000 5250 50  0001 C CNN
+F 0 "#PWR2" H 1000 5250 50  0001 C CNN
 F 1 "+3.3V" H 1000 5540 50  0000 C CNN
 F 2 "" H 1000 5400 50  0001 C CNN
@@
 $EndComp
 $Comp
-L GND #PWR013
+L GND #PWR3
 U 1 1 5B182781
 P 1000 5900
-F 0 "#PWR013" H 1000 5650 50  0001 C CNN
+F 0 "#PWR3" H 1000 5650 50  0001 C CNN
 F 1 "GND" H 1000 5750 50  0000 C CNN
 F 2 "" H 1000 5900 50  0001 C CNN
@@
 Wire Wire Line
 	1000 5800 1000 5900
-$Comp
-L Crystal Y1
-U 1 1 5B1829A5
-P 4800 5300
-F 0 "Y1" H 4800 5450 50  0000 C CNN
-F 1 "16MHz" H 4800 5150 50  0000 C CNN
-F 2 "Crystals:Crystal_SMD_0603-4pin_6.0x3.5mm_HandSoldering" H 4800 5300 50  0001 C CNN
-F 3 "" H 4800 5300 50  0001 C CNN
-	1    4800 5300
-	0    1    1    0
-$EndComp
-Wire Wire Line
-	4350 5500 5000 5500
-Wire Wire Line
-	4800 5500 4800 5450
 $Comp
 L R R4
@@
 	4350 5250 4350 5100
 Wire Wire Line
-	4350 5100 5000 5100
-Wire Wire Line
 	4450 5100 4450 5150
-Wire Wire Line
-	4800 5100 4800 5150
 Connection ~ 4450 5100
 Wire Wire Line
@@
 L C C2
 U 1 1 5B1832F7
-P 5150 5100
-F 0 "C2" V 5200 5200 50  0000 L CNN
-F 1 "22pF" V 5200 4850 50  0000 L CNN
-F 2 "Capacitors_SMD:C_0603_HandSoldering" H 5188 4950 50  0001 C CNN
-F 3 "" H 5150 5100 50  0001 C CNN
-	1    5150 5100
+P 5450 5100
+F 0 "C2" V 5500 5200 50  0000 L CNN
+F 1 "22pF" V 5500 4850 50  0000 L CNN
+F 2 "Capacitors_SMD:C_0603_HandSoldering" H 5488 4950 50  0001 C CNN
+F 3 "" H 5450 5100 50  0001 C CNN
+	1    5450 5100
 	0    -1   -1   0
 $EndComp
@@
 L C C3
 U 1 1 5B18344D
-P 5150 5500
-F 0 "C3" V 5200 5600 50  0000 L CNN
-F 1 "22pF" V 5200 5250 50  0000 L CNN
-F 2 "Capacitors_SMD:C_0603_HandSoldering" H 5188 5350 50  0001 C CNN
-F 3 "" H 5150 5500 50  0001 C CNN
-	1    5150 5500
+P 5450 5500
+F 0 "C3" V 5500 5600 50  0000 L CNN
+F 1 "22pF" V 5500 5250 50  0000 L CNN
+F 2 "Capacitors_SMD:C_0603_HandSoldering" H 5488 5350 50  0001 C CNN
+F 3 "" H 5450 5500 50  0001 C CNN
+	1    5450 5500
 	0    -1   -1   0
 $EndComp
-Connection ~ 4800 5100
-Connection ~ 4800 5500
-$Comp
-L GND #PWR014
+$Comp
+L GND #PWR13
 U 1 1 5B18359F
-P 5450 5600
-F 0 "#PWR014" H 5450 5350 50  0001 C CNN
-F 1 "GND" H 5450 5450 50  0000 C CNN
-F 2 "" H 5450 5600 50  0001 C CNN
-F 3 "" H 5450 5600 50  0001 C CNN
-	1    5450 5600
-	1    0    0    -1
-$EndComp
-Wire Wire Line
-	5300 5100 5450 5100
-Wire Wire Line
-	5450 5100 5450 5600
-Wire Wire Line
-	5300 5500 5450 5500
-Connection ~ 5450 5500
+P 5750 5600
+F 0 "#PWR13" H 5750 5350 50  0001 C CNN
+F 1 "GND" H 5750 5450 50  0000 C CNN
+F 2 "" H 5750 5600 50  0001 C CNN
+F 3 "" H 5750 5600 50  0001 C CNN
+	1    5750 5600
+	1    0    0    -1
+$EndComp
+Wire Wire Line
+	5600 5100 5750 5100
+Wire Wire Line
+	5750 5100 5750 5600
+Wire Wire Line
+	5750 5500 5600 5500
 $Comp
 L R R3
@@
 $EndComp
 $Comp
-L +3.3V #PWR015
+L +3.3V #PWR10
 U 1 1 5B18394F
 P 4350 5750
-F 0 "#PWR015" H 4350 5600 50  0001 C CNN
+F 0 "#PWR10" H 4350 5600 50  0001 C CNN
 F 1 "+3.3V" H 4350 5890 50  0000 C CNN
 F 2 "" H 4350 5750 50  0001 C CNN
@@
 	4350 5750 4350 5800
 $Comp
-L +3.3V #PWR016
+L +3.3V #PWR4
 U 1 1 5B183D8D
 P 1600 2550
-F 0 "#PWR016" H 1600 2400 50  0001 C CNN
+F 0 "#PWR4" H 1600 2400 50  0001 C CNN
 F 1 "+3.3V" H 1600 2690 50  0000 C CNN
 F 2 "" H 1600 2550 50  0001 C CNN
@@
 $EndComp
 $Comp
-L GND #PWR017
+L GND #PWR5
 U 1 1 5B183DD4
 P 1600 3550
-F 0 "#PWR017" H 1600 3300 50  0001 C CNN
+F 0 "#PWR5" H 1600 3300 50  0001 C CNN
 F 1 "GND" H 1600 3400 50  0000 C CNN
 F 2 "" H 1600 3550 50  0001 C CNN
@@
 $EndComp
 $Comp
-L GND #PWR018
+L GND #PWR9
 U 1 1 5B1855B3
 P 2850 3350
-F 0 "#PWR018" H 2850 3100 50  0001 C CNN
+F 0 "#PWR9" H 2850 3100 50  0001 C CNN
 F 1 "GND" H 2850 3200 50  0000 C CNN
 F 2 "" H 2850 3350 50  0001 C CNN
@@
 $EndComp
 $Comp
-L GND #PWR019
+L GND #PWR16
 U 1 1 5B18665A
 P 7450 4950
-F 0 "#PWR019" H 7450 4700 50  0001 C CNN
+F 0 "#PWR16" H 7450 4700 50  0001 C CNN
 F 1 "GND" H 7450 4800 50  0000 C CNN
 F 2 "" H 7450 4950 50  0001 C CNN
@@
 	7450 4300 7800 4300
 Connection ~ 7450 4300
+NoConn ~ 1100 6450
+NoConn ~ 1100 6550
+NoConn ~ 1100 6650
+NoConn ~ 1100 6750
+NoConn ~ 3700 7050
+NoConn ~ 3700 6950
+NoConn ~ 3700 6850
+NoConn ~ 3700 6750
+NoConn ~ 3700 6550
+NoConn ~ 3700 6450
+NoConn ~ 3700 6350
+Wire Wire Line
+	3700 4750 4200 4750
+Text Label 4200 4750 2    60   ~ 0
+D9
+Wire Wire Line
+	3700 5750 4200 5750
+Wire Wire Line
+	3700 5850 4200 5850
+Wire Wire Line
+	3700 5950 4200 5950
+Wire Wire Line
+	3700 6050 4200 6050
+NoConn ~ 4200 5750
+NoConn ~ 4200 5850
+NoConn ~ 4200 5950
+NoConn ~ 4200 6050
+Text Label 4700 1150 0    60   ~ 0
+D9
+$Comp
+L Crystal_GND24 Y1
+U 1 1 5B211C62
+P 5000 5300
+F 0 "Y1" V 4750 5150 50  0000 L CNN
+F 1 "Crystal_GND24" V 5250 5050 50  0000 L CNN
+F 2 "Crystals:Crystal_SMD_3225-4pin_3.2x2.5mm_HandSoldering" H 5000 5300 50  0001 C CNN
+F 3 "" H 5000 5300 50  0001 C CNN
+	1    5000 5300
+	0    1    1    0
+$EndComp
+Wire Wire Line
+	4350 5100 5300 5100
+Wire Wire Line
+	4350 5500 5300 5500
+$Comp
+L GND #PWR11
+U 1 1 5B212244
+P 4700 5300
+F 0 "#PWR11" H 4700 5050 50  0001 C CNN
+F 1 "GND" H 4700 5150 50  0000 C CNN
+F 2 "" H 4700 5300 50  0001 C CNN
+F 3 "" H 4700 5300 50  0001 C CNN
+	1    4700 5300
+	1    0    0    -1
+$EndComp
+Connection ~ 5750 5500
+Wire Wire Line
+	5000 5500 5000 5450
+Connection ~ 5000 5500
+Wire Wire Line
+	5000 5150 5000 5100
+Connection ~ 5000 5100
+Wire Wire Line
+	4800 5300 4700 5300
+Wire Wire Line
+	5200 5300 5750 5300
+Connection ~ 5750 5300
+$Comp
+L Conn_01x01 J4
+U 1 1 5B212E6E
+P 10250 2400
+F 0 "J4" H 10250 2500 50  0000 C CNN
+F 1 "MECH" H 10250 2300 50  0000 C CNN
+F 2 "Mounting_Holes:MountingHole_5.3mm_M5" H 10250 2400 50  0001 C CNN
+F 3 "" H 10250 2400 50  0001 C CNN
+	1    10250 2400
+	1    0    0    -1
+$EndComp
+NoConn ~ 10050 2400
 $EndSCHEMATC
